Commit message: Fix ovis joints based on testing in rviz

File: src/ovis_description/urdf/ovis.urdf.xacro (robot description, xacro)
@@ -38,5 +38,5 @@
     <xacro:property name="joint_1" value="joint_1" />
     <xacro:property name="joint_1_type" value="continuous" />
-    <xacro:property name="joint_1_axis_xyz" value="0 0 1" />
+    <xacro:property name="joint_1_axis_xyz" value="0 1 0" />
     <xacro:property name="joint_1_origin_xyz" value="0 0.051 0" />
     <xacro:property name="joint_1_origin_rpy" value="0 0 0" />
@@ -49,5 +49,5 @@
     <xacro:property name="joint_2_axis_xyz" value="0 0 1" />
     <xacro:property name="joint_2_origin_xyz" value="0 0.0889 0" />
-    <xacro:property name="joint_2_origin_rpy" value="0 0 ${J_PI/2}" />
+    <xacro:property name="joint_2_origin_rpy" value="0 0 0" />
     <xacro:property name="joint_2_lower_limit" value="${-J_PI/2}" />
     <xacro:property name="joint_2_upper_limit" value="${J_PI/2}" />

Commit message: Transferred base point to a xacro parameter so it can be inserted in the right spot on the robot

File: src/ovis_description/urdf/ovis.urdf.xacro (robot description, xacro)
@@ -34,5 +34,6 @@
     <xacro:property name="joint_base_type" value="fixed" />
     <xacro:property name="joint_base_axis_xyz" value="0 0 0" />
-    <xacro:property name="joint_base_origin_xyz" value="0 0 0" />
+    <!-- Transferred to a parameter in the ovis macro -->
+    <!-- <xacro:property name="joint_base_origin_xyz" value="0 0 0" /> -->
     <xacro:property name="joint_base_origin_rpy" value="${J_PI/2} 0 0" />
     <xacro:property name="joint_1" value="joint_1" />
@@ -97,5 +98,5 @@
     <xacro:property name="joint_end_effector_origin_xyz" value="0 0 -0.1600" />
     <xacro:property name="joint_end_effector_origin_rpy" value="${J_PI} 0 ${J_PI/2}" />
-    <xacro:macro name="ovis" params="base_parent prefix:=ovis">
+    <xacro:macro name="ovis" params="base_parent prefix:=ovis joint_base_origin_xyz:='0 0 0'">
         <xacro:gazebo_config robot_namespace="${prefix}" />
         <xacro:kinova_armlink link_name="${prefix}_link_base" link_mesh="${link_base_mesh}"

Commit message: Update joint limits and start positions in ovis.urdf.xacro

File: src/ovis_description/urdf/ovis.urdf.xacro (robot description, xacro)
@@ -50,7 +50,7 @@
     <xacro:property name="joint_2_axis_xyz" value="0 0 1" />
     <xacro:property name="joint_2_origin_xyz" value="0 0.0889 0" />
-    <xacro:property name="joint_2_origin_rpy" value="0 0 0" />
-    <xacro:property name="joint_2_lower_limit" value="${-J_PI/2}" />
-    <xacro:property name="joint_2_upper_limit" value="${J_PI/2}" />
+    <xacro:property name="joint_2_origin_rpy" value="0 0 ${-J_PI/2}" />
+    <xacro:property name="joint_2_lower_limit" value="0" />
+    <xacro:property name="joint_2_upper_limit" value="${J_PI}" />
     <xacro:property name="joint_2_velocity_limit" value="${36*J_PI/180}" />
     <xacro:property name="joint_2_torque_limit" value="80" />
@@ -59,7 +59,7 @@
     <xacro:property name="joint_3_axis_xyz" value="0 0 1" />
     <xacro:property name="joint_3_origin_xyz" value="0 0.465 0" />
-    <xacro:property name="joint_3_origin_rpy" value="0 0 ${J_PI/2}" />
-    <xacro:property name="joint_3_lower_limit" value="${-J_PI/2}" />
-    <xacro:property name="joint_3_upper_limit" value="${J_PI/2}" />
+    <xacro:property name="joint_3_origin_rpy" value="0 0 ${J_PI}" />
+    <xacro:property name="joint_3_lower_limit" value="${-J_PI}" />
+    <xacro:property name="joint_3_upper_limit" value="0" />
     <xacro:property name="joint_3_velocity_limit" value="${36*J_PI/180}" />
     <xacro:property name="joint_3_torque_limit" value="40" />
