Commit message: Changed the values for the dimensions and axis of Ovis

File: src/ovis_description/urdf/kinova_common.xacro (robot description, xacro)
@@ -20,8 +20,8 @@
                 <geometry>
                     <mesh
-                        filename="package://ovis_description/meshes/${link_mesh}.STL"/>
+                        filename="$(find ovis_description)/meshes/${link_mesh}.stl"/>
                 </geometry>
                 <material name="carbon_fiber">
-                    <color rgba="0.792156862745098 0.819607843137255 0.933333333333333 1" />
+                    <color rgba="0.792156862745098 0 0 1" />
                 </material>
             </visual>
@@ -31,5 +31,5 @@
                 <geometry>
                     <mesh
-                        filename="package://ovis_description/meshes/${ring_mesh}.STL"/>
+                        filename="$(find ovis_description)/meshes/${ring_mesh}.stl"/>
                 </geometry>
              </visual>
@@ -38,5 +38,5 @@
                 <geometry>
                     <mesh
-                        filename="package://ovis_description/meshes/${link_mesh}.STL"/>
+                        filename="$(find ovis_description)/meshes/${link_mesh}.stl"/>
                 </geometry>
             </collision>

File: src/ovis_description/urdf/ovis.urdf.xacro (robot description, xacro)
@@ -17,11 +17,11 @@
     <!-- Import all Gazebo-customization elements -->
     <xacro:include filename="$(find ovis_description)/urdf/ovis.gazebo" />
-    <xacro:property name="link_base_mesh" value="base" />
-    <xacro:property name="link_1_mesh" value="shoulder" />
-    <xacro:property name="link_2_mesh" value="arm" />
-    <xacro:property name="link_3_mesh" value="forearm" />
-    <xacro:property name="link_4_mesh" value="wrist" />
-    <xacro:property name="link_5_mesh" value="wrist" />
-    <xacro:property name="link_6_mesh" value="hand_3finger" />
+    <xacro:property name="link_base_mesh" value="visual/ovis_base" />
+    <xacro:property name="link_1_mesh" value="visual/ovis_shoulder" />
+    <xacro:property name="link_2_mesh" value="visual/ovis_upper_arm" />
+    <xacro:property name="link_3_mesh" value="visual/ovis_elbow" />
+    <xacro:property name="link_4_mesh" value="visual/ovis_forearm" />
+    <xacro:property name="link_5_mesh" value="visual/ovis_wrist" />
+    <xacro:property name="link_6_mesh" value="visual/ovis_flange" />
     <xacro:property name="link_base_mesh_no" value="0" />
     <xacro:property name="link_1_mesh_no" value="1" />
@@ -35,12 +35,12 @@
     <xacro:property name="joint_base_axis_xyz" value="0 0 0" />
     <xacro:property name="joint_base_origin_xyz" value="0 0 0" />
-    <xacro:property name="joint_base_origin_rpy" value="0 0 0" />
+    <xacro:property name="joint_base_origin_rpy" value="${J_PI/2} 0 0" />
     <xacro:property name="joint_1" value="joint_1" />
     <xacro:property name="joint_1_type" value="continuous" />
     <xacro:property name="joint_1_axis_xyz" value="0 0 1" />
-    <xacro:property name="joint_1_origin_xyz" value="0 0 0.15675" />
-    <xacro:property name="joint_1_origin_rpy" value="0 ${J_PI} 0" />
-    <xacro:property name="joint_1_lower_limit" value="${-2*J_PI}" />
-    <xacro:property name="joint_1_upper_limit" value="${2*J_PI}" />
+    <xacro:property name="joint_1_origin_xyz" value="0 0.051 0" />
+    <xacro:property name="joint_1_origin_rpy" value="0 0 0" />
+    <xacro:property name="joint_1_lower_limit" value="${-4*J_PI}" />
+    <xacro:property name="joint_1_upper_limit" value="${4*J_PI}" />
     <xacro:property name="joint_1_velocity_limit" value="${36*J_PI/180}" />
     <xacro:property name="joint_1_torque_limit" value="40" />
@@ -48,8 +48,8 @@
     <xacro:property name="joint_2_type" value="revolute" />
     <xacro:property name="joint_2_axis_xyz" value="0 0 1" />
-    <xacro:property name="joint_2_origin_xyz" value="0 0.0016 -0.11875" />
-    <xacro:property name="joint_2_origin_rpy" value="-${J_PI/2} 0 ${J_PI}" />
-    <xacro:property name="joint_2_lower_limit" value="${47/180*J_PI}" />
-    <xacro:property name="joint_2_upper_limit" value="${313/180*J_PI}" />
+    <xacro:property name="joint_2_origin_xyz" value="0 0.0889 0" />
+    <xacro:property name="joint_2_origin_rpy" value="0 0 ${J_PI/2}" />
+    <xacro:property name="joint_2_lower_limit" value="${-J_PI/2}" />
+    <xacro:property name="joint_2_upper_limit" value="${J_PI/2}" />
     <xacro:property name="joint_2_velocity_limit" value="${36*J_PI/180}" />
     <xacro:property name="joint_2_torque_limit" value="80" />
@@ -57,26 +57,26 @@
     <xacro:property name="joint_3_type" value="revolute" />
     <xacro:property name="joint_3_axis_xyz" value="0 0 1" />
-    <xacro:property name="joint_3_origin_xyz" value="0 -0.410 0" />
-    <xacro:property name="joint_3_origin_rpy" value="0 ${J_PI} 0" />
-    <xacro:property name="joint_3_lower_limit" value="${19/180*J_PI}" />
-    <xacro:property name="joint_3_upper_limit" value="${341/180*J_PI}" />
+    <xacro:property name="joint_3_origin_xyz" value="0 0.465 0" />
+    <xacro:property name="joint_3_origin_rpy" value="0 0 ${J_PI/2}" />
+    <xacro:property name="joint_3_lower_limit" value="${-J_PI/2}" />
+    <xacro:property name="joint_3_upper_limit" value="${J_PI/2}" />
     <xacro:property name="joint_3_velocity_limit" value="${36*J_PI/180}" />
     <xacro:property name="joint_3_torque_limit" value="40" />
     <xacro:property name="joint_4" value="joint_4" />
     <xacro:property name="joint_4_type" value="continuous" />
-    <xacro:property name="joint_4_axis_xyz" value="0 0 1" />
-    <xacro:property name="joint_4_origin_xyz" value="0 0.2073 -0.0114" />
-    <xacro:property name="joint_4_origin_rpy" value="-${J_PI/2} 0 ${J_PI}" />
-    <xacro:property name="joint_4_lower_limit" value="${-2*J_PI}" />
-    <xacro:property name="joint_4_upper_limit" value="${2*J_PI}" />
+    <xacro:property name="joint_4_axis_xyz" value="0 1 0" />
+    <xacro:property name="joint_4_origin_xyz" value="0.0889 0.047625 0" />
+    <xacro:property name="joint_4_origin_rpy" value="0 0 0" />
+    <xacro:property name="joint_4_lower_limit" value="${-4*J_PI}" />
+    <xacro:property name="joint_4_upper_limit" value="${4*J_PI}" />
     <xacro:property name="joint_4_velocity_limit" value="${48*J_PI/180}" />
     <xacro:property name="joint_4_torque_limit" value="20" />
     <xacro:property name="joint_5" value="joint_5" />
-    <xacro:property name="joint_5_type" value="continuous" />
+    <xacro:property name="joint_5_type" value="revolute" />
     <xacro:property name="joint_5_axis_xyz" value="0 0 1" />
-    <xacro:property name="joint_5_origin_xyz" value="0 -0.03703 -0.06414" />
-    <xacro:property name="joint_5_origin_rpy" value="${J_PI/3} 0 ${J_PI}" />
-    <xacro:property name="joint_5_lower_limit" value="${-2*J_PI}" />
-    <xacro:property name="joint_5_upper_limit" value="${2*J_PI}" />
+    <xacro:property name="joint_5_origin_xyz" value="0 0.265 0" />
+    <xacro:property name="joint_5_origin_rpy" value="0 0 0" />
+    <xacro:property name="joint_5_lower_limit" value="${-J_PI/2}" />
+    <xacro:property name="joint_5_upper_limit" value="${J_PI/2}" />
     <xacro:property name="joint_5_velocity_limit" value="${48*J_PI/180}" />
     <xacro:property name="joint_5_torque_limit" value="20" />
@@ -84,6 +84,6 @@
     <xacro:property name="joint_6_type" value="continuous" />
     <xacro:property name="joint_6_axis_xyz" value="0 0 1" />
-    <xacro:property name="joint_6_origin_xyz" value="0 -0.03703 -0.06414" />
-    <xacro:property name="joint_6_origin_rpy" value="${J_PI/3} 0 ${J_PI}" />
+    <xacro:property name="joint_6_origin_xyz" value="0 0.0762 0" />
+    <xacro:property name="joint_6_origin_rpy" value="${J_PI/2} ${J_PI/2} 0" />
     <!-- If gripper inverted, use this line instead -->
     <!-- <xacro:property name="joint_6_origin_rpy" value="$${-J_PI/3} 0 0" /> -->
@@ -107,5 +107,5 @@
             joint_velocity_limit="0" joint_torque_limit="0" fixed="true" />
         <xacro:kinova_armlink link_name="${prefix}_link_1" link_mesh="${link_1_mesh}"
-            use_ring_mesh="true" mesh_no="${link_1_mesh_no}" />
+            use_ring_mesh="false" mesh_no="${link_1_mesh_no}" />
         <xacro:kinova_armjoint joint_name="${prefix}_joint_1" type="${joint_1_type}"
             parent="${prefix}_link_base" child="${prefix}_link_1"
@@ -116,5 +116,5 @@
             joint_torque_limit="${joint_1_torque_limit}" />
         <xacro:kinova_armlink link_name="${prefix}_link_2" link_mesh="${link_2_mesh}"
-            use_ring_mesh="true" mesh_no="${link_2_mesh_no}" />
+            use_ring_mesh="false" mesh_no="${link_2_mesh_no}" />
         <xacro:kinova_armjoint joint_name="${prefix}_joint_2" type="${joint_2_type}"
             parent="${prefix}_link_1" child="${prefix}_link_2" joint_axis_xyz="${joint_2_axis_xyz}"
@@ -124,5 +124,5 @@
             joint_torque_limit="${joint_2_torque_limit}" />
         <xacro:kinova_armlink link_name="${prefix}_link_3" link_mesh="${link_3_mesh}"
-            use_ring_mesh="true" mesh_no="${link_3_mesh_no}" />
+            use_ring_mesh="false" mesh_no="${link_3_mesh_no}" />
         <xacro:kinova_armjoint joint_name="${prefix}_joint_3" type="${joint_3_type}"
             parent="${prefix}_link_2" child="${prefix}_link_3" joint_axis_xyz="${joint_3_axis_xyz}"
@@ -132,5 +132,5 @@
             joint_torque_limit="${joint_3_torque_limit}" />
         <xacro:kinova_armlink link_name="${prefix}_link_4" link_mesh="${link_4_mesh}"
-            use_ring_mesh="true" ring_mesh="ring_small" mesh_no="${link_4_mesh_no}" />
+            use_ring_mesh="false" ring_mesh="ring_small" mesh_no="${link_4_mesh_no}" />
         <xacro:kinova_armjoint joint_name="${prefix}_joint_4" type="${joint_4_type}"
             parent="${prefix}_link_3" child="${prefix}_link_4" joint_axis_xyz="${joint_4_axis_xyz}"
@@ -140,5 +140,5 @@
             joint_torque_limit="${joint_4_torque_limit}" />
         <xacro:kinova_armlink link_name="${prefix}_link_5" link_mesh="${link_5_mesh}"
-            use_ring_mesh="true" ring_mesh="ring_small" mesh_no="${link_5_mesh_no}" />
+            use_ring_mesh="false" ring_mesh="ring_small" mesh_no="${link_5_mesh_no}" />
         <xacro:kinova_armjoint joint_name="${prefix}_joint_5" type="${joint_5_type}"
             parent="${prefix}_link_4" child="${prefix}_link_5" joint_axis_xyz="${joint_5_axis_xyz}"
@@ -148,5 +148,5 @@
             joint_torque_limit="${joint_5_torque_limit}" />
         <xacro:kinova_armlink link_name="${prefix}_link_6" link_mesh="${link_6_mesh}"
-            use_ring_mesh="true" ring_mesh="ring_small" mesh_no="${link_6_mesh_no}" />
+            use_ring_mesh="false" ring_mesh="ring_small" mesh_no="${link_6_mesh_no}" />
         <xacro:kinova_armjoint joint_name="${prefix}_joint_6" type="${joint_6_type}"
             parent="${prefix}_link_5" child="${prefix}_link_6" joint_axis_xyz="${joint_6_axis_xyz}"
@@ -164,40 +164,3 @@
         <!-- <xacro:kinova_3fingers link_hand="${prefix}_link_6" prefix="${prefix}_"/> -->
     </xacro:macro>
-    <!-- <material name="rubber_color">
-    <color rgba="0.1 0.1 0.1 1.0"/>
-</material>
-<material name="frame_color">
-    <color rgba="0.5 0.5 0.5 1.0"/>
-</material>
-<material name="lidar_color">
-    <color rgba="1 0 0 1.0"/>
-</material>
-<xacro:include filename="$(find ovis_description)/urdf/gazebo.urdf.xacro" />
-<xacro:include filename="$(find ovis_description)/urdf/imu.urdf.xacro" />
-<link name="base_footprint"/> -->
-    <!-- <link name="base_link">
-        <visual>
-            <origin xyz="0 0 0" rpy="0 0 0"/>
-            <geometry>
-                <mesh filename="file://$(find ovis_description)/meshes/base.stl"/>
-            </geometry>
-            <material name="frame_color"/>
-        </visual>
-        <collision>
-            <origin xyz="0 0 0" rpy="0 0 0"/>
-            <geometry>
-                <mesh filename="file://$(find ovis_description)/meshes/base.stl"/>
-            </geometry>
-        </collision>
-        <inertial>
-            <origin xyz="0 0 0.5" rpy="0 0 0"/>
-            <mass value="80"/>
-            <inertia ixx="100"  ixy="0"  ixz="0" iyy="100" iyz="0" izz="100" />
-        </inertial>
-    </link>
-    <joint name="base_joint" type="fixed">
-        <origin rpy="0 0 0" xyz="0 0 0"/>
-        <parent link="base_footprint"/>
-        <child link="base_link"/>
-    </joint> -->
 </root>

Commit message: Fix Rviz sim by using the names it wants and it's file path resolving by changing a detail in kinova libs

File: src/ovis_description/urdf/kinova_common.xacro (robot description, xacro)
@@ -20,5 +20,5 @@
                 <geometry>
                     <mesh
-                        filename="$(find ovis_description)/meshes/${link_mesh}.stl"/>
+                        filename="file://$(find ovis_description)/meshes/${link_mesh}.stl"/>
                 </geometry>
                 <material name="carbon_fiber">

File: src/ovis_description/urdf/ovis_standalone.urdf.xacro (robot description, xacro)
@@ -14,13 +14,13 @@
     xmlns:xacro="http://www.ros.org/wiki/xacro" name="ovis">
     <xacro:include filename="$(find ovis_description)/urdf/ovis.urdf.xacro" />
-    <link name="root" />
+    <link name="base_link" />
     <!-- for gazebo -->
-    <link name="world" />
-    <joint name="connect_root_and_world" type="fixed">
+    <!-- <link name="world" /> -->
+    <!-- <joint name="connect_root_and_world" type="fixed">
         <child link="root" />
         <parent link="world" />
         <origin xyz="0 0 0" rpy="0 0 0" />
-    </joint>
-    <xacro:property name="robot_root" value="root" />
+    </joint> -->
+    <xacro:property name="robot_root" value="base_link" />
     <xacro:ovis base_parent="${robot_root}" />
 </robot>

Commit message: fix collision files not being loaded

File: src/ovis_description/urdf/kinova_common.xacro (robot description, xacro)
@@ -20,5 +20,5 @@
                 <geometry>
                     <mesh
-                        filename="file://$(find ovis_description)/meshes/${link_mesh}.stl"/>
+                        filename="file://$(find ovis_description)/meshes/visual/${link_mesh}.stl"/>
                 </geometry>
                 <material name="carbon_fiber">
@@ -34,9 +34,9 @@
                 </geometry>
              </visual>
-	    </xacro:if>
+	          </xacro:if>
             <collision>
                 <geometry>
                     <mesh
-                        filename="$(find ovis_description)/meshes/${link_mesh}.stl"/>
+                        filename="file://$(find ovis_description)/meshes/collision/${link_mesh}.stl"/>
                 </geometry>
             </collision>

File: src/ovis_description/urdf/ovis.urdf.xacro (robot description, xacro)
@@ -17,11 +17,11 @@
     <!-- Import all Gazebo-customization elements -->
     <xacro:include filename="$(find ovis_description)/urdf/ovis.gazebo" />
-    <xacro:property name="link_base_mesh" value="visual/ovis_base" />
-    <xacro:property name="link_1_mesh" value="visual/ovis_shoulder" />
-    <xacro:property name="link_2_mesh" value="visual/ovis_upper_arm" />
-    <xacro:property name="link_3_mesh" value="visual/ovis_elbow" />
-    <xacro:property name="link_4_mesh" value="visual/ovis_forearm" />
-    <xacro:property name="link_5_mesh" value="visual/ovis_wrist" />
-    <xacro:property name="link_6_mesh" value="visual/ovis_flange" />
+    <xacro:property name="link_base_mesh" value="ovis_base" />
+    <xacro:property name="link_1_mesh" value="ovis_shoulder" />
+    <xacro:property name="link_2_mesh" value="ovis_upper_arm" />
+    <xacro:property name="link_3_mesh" value="ovis_elbow" />
+    <xacro:property name="link_4_mesh" value="ovis_forearm" />
+    <xacro:property name="link_5_mesh" value="ovis_wrist" />
+    <xacro:property name="link_6_mesh" value="ovis_flange" />
     <xacro:property name="link_base_mesh_no" value="0" />
     <xacro:property name="link_1_mesh_no" value="1" />
