Commit message: add basic moveit config

File: src/ovis_description/urdf/gazebo.urdf.xacro (robot description, xacro)
@@ -4,5 +4,5 @@
         <!-- ros_control plugin -->
         <gazebo>
-            <plugin name="gazebo_ros_control" filename="libgazebo_ros_control.so">
+            <plugin name="gazebo_ros_control" filename="gz_ros_control.so">
                 <robotNamespace>${robot_namespace}</robotNamespace>
                 <robotSimType>gazebo_ros_control/DefaultRobotHWSim</robotSimType>

File: src/ovis_description/urdf/kinova_common.xacro (robot description, xacro)
@@ -103,5 +103,5 @@
       </gazebo>
       <gazebo>
-        <plugin name="ft_sensor" filename="libgazebo_ros_ft_sensor.so">
+        <plugin name="ft_sensor" filename="gz_ros_ft_sensor.so">
           <updateRate>30.0</updateRate>
           <topicName>${joint_name}_ft_sensor_topic</topicName>

File: src/ovis_description/urdf/ovis.urdf.xacro (robot description, xacro)
@@ -1,20 +1,4 @@
 <?xml version="1.0"?>
-<root xmlns:xi="http://www.w3.org/2001/XInclude"
-    xmlns:gazebo="http://playerstage.sourceforge.net/gazebo/xmlschema/#gz"
-    xmlns:model="http://playerstage.sourceforge.net/gazebo/xmlschema/#model"
-    xmlns:sensor="http://playerstage.sourceforge.net/gazebo/xmlschema/#sensor"
-    xmlns:body="http://playerstage.sourceforge.net/gazebo/xmlschema/#body"
-    xmlns:geom="http://playerstage.sourceforge.net/gazebo/xmlschema/#geom"
-    xmlns:joint="http://playerstage.sourceforge.net/gazebo/xmlschema/#joint"
-    xmlns:controller="http://playerstage.sourceforge.net/gazebo/xmlschema/#controller"
-    xmlns:interface="http://playerstage.sourceforge.net/gazebo/xmlschema/#interface"
-    xmlns:rendering="http://playerstage.sourceforge.net/gazebo/xmlschema/#rendering"
-    xmlns:renderable="http://playerstage.sourceforge.net/gazebo/xmlschema/#renderable"
-    xmlns:physics="http://playerstage.sourceforge.net/gazebo/xmlschema/#physics"
-    xmlns:xacro="http://www.ros.org/wiki/xacro">
-    <xacro:include filename="$(find ovis_description)/urdf/kinova_common.xacro" />
-    <!-- <xacro:include filename="$(find ovis_description)/urdf/kinova_finger_set.xacro" /> -->
-    <!-- Import all Gazebo-customization elements -->
-    <xacro:include filename="$(find ovis_description)/urdf/gazebo.urdf.xacro" />
+<root xmlns:xacro="http://www.ros.org/wiki/xacro">
     <xacro:property name="link_base_mesh" value="visual/ovis_base" />
     <xacro:property name="link_1_mesh" value="visual/ovis_shoulder" />
@@ -163,5 +147,4 @@
             joint_origin_rpy="${joint_end_effector_origin_rpy}" joint_lower_limit="0"
             joint_upper_limit="0" />
-        <!-- <xacro:kinova_3fingers link_hand="${prefix}_link_6" prefix="${prefix}_"/> -->
     </xacro:macro>
 </root>

File: src/ovis_description/urdf/ovis_standalone.urdf.xacro (robot description, xacro)
@@ -1,25 +1,8 @@
 <?xml version="1.0"?>
-<robot xmlns:xi="http://www.w3.org/2001/XInclude"
-    xmlns:gazebo="http://playerstage.sourceforge.net/gazebo/xmlschema/#gz"
-    xmlns:model="http://playerstage.sourceforge.net/gazebo/xmlschema/#model"
-    xmlns:sensor="http://playerstage.sourceforge.net/gazebo/xmlschema/#sensor"
-    xmlns:body="http://playerstage.sourceforge.net/gazebo/xmlschema/#body"
-    xmlns:geom="http://playerstage.sourceforge.net/gazebo/xmlschema/#geom"
-    xmlns:joint="http://playerstage.sourceforge.net/gazebo/xmlschema/#joint"
-    xmlns:controller="http://playerstage.sourceforge.net/gazebo/xmlschema/#controller"
-    xmlns:interface="http://playerstage.sourceforge.net/gazebo/xmlschema/#interface"
-    xmlns:rendering="http://playerstage.sourceforge.net/gazebo/xmlschema/#rendering"
-    xmlns:renderable="http://playerstage.sourceforge.net/gazebo/xmlschema/#renderable"
-    xmlns:physics="http://playerstage.sourceforge.net/gazebo/xmlschema/#physics"
-    xmlns:xacro="http://www.ros.org/wiki/xacro" name="ovis">
+<robot name="ovis" xmlns:xacro="http://www.ros.org/wiki/xacro">
+    <xacro:include filename="$(find ovis_description)/urdf/gazebo.urdf.xacro" />
     <xacro:include filename="$(find ovis_description)/urdf/ovis.urdf.xacro" />
+    <xacro:include filename="$(find ovis_description)/urdf/kinova_common.xacro" />
     <link name="base_link" />
-    <!-- for gazebo -->
-    <!-- <link name="world" /> -->
-    <!-- <joint name="connect_root_and_world" type="fixed">
-        <child link="root" />
-        <parent link="world" />
-        <origin xyz="0 0 0" rpy="0 0 0" />
-    </joint> -->
     <xacro:property name="robot_root" value="base_link" />
     <xacro:ovis base_parent="${robot_root}" />

Commit message: remove need for gazebo_config

File: src/ovis_description/urdf/gazebo.urdf.xacro (robot description, xacro)
@@ -1,16 +1,14 @@
 <?xml version="1.0"?>
 <robot xmlns:xacro="http://www.ros.org/wiki/xacro">
-    <xacro:macro name="gazebo_config" params="robot_namespace">
-        <!-- ros_control plugin -->
-        <gazebo>
-            <plugin filename="gz_ros2_control-system"
-                name="gz_ros2_control::GazeboSimROS2ControlPlugin">
-                <robot_param>robot_description</robot_param>
-                <robot_param_node>robot_state_publisher</robot_param_node>
-                <parameters>$(find ovis_moveit)/config/ros2_controllers.yaml</parameters>
-                <controller_manager_prefix_node_name>controller_manager</controller_manager_prefix_node_name>
-            </plugin>
-        </gazebo>
-    </xacro:macro>
+    <!-- ros_control plugin -->
+    <gazebo>
+        <plugin filename="gz_ros2_control-system"
+            name="gz_ros2_control::GazeboSimROS2ControlPlugin">
+            <robot_param>robot_description</robot_param>
+            <robot_param_node>robot_state_publisher</robot_param_node>
+            <parameters>$(find ovis_moveit)/config/ros2_controllers.yaml</parameters>
+            <controller_manager_prefix_node_name>controller_manager</controller_manager_prefix_node_name>
+        </plugin>
+    </gazebo>
     <gazebo>
         <plugin

Commit message: trajectory planner support with rove

File: src/ovis_description/urdf/gazebo.urdf.xacro (robot description, xacro)
@@ -14,15 +14,3 @@
         </plugin>
     </gazebo>
-    <gazebo>
-        <plugin
-            filename="gz-sim-joint-state-publisher-system"
-            name="gz::sim::systems::JointStatePublisher">
-            <topic>joint_states</topic>
-        </plugin>
-         <plugin
-            filename="gz-sim-sensors-system"
-            name="gz::sim::systems::Sensors">
-            <render_engine>ogre2</render_engine>
-        </plugin>
-    </gazebo>
 </robot>

File: src/ovis_description/urdf/ovis2/urdf/ovis_standalone.urdf.xacro (robot description, xacro)
@@ -4,6 +4,6 @@
     <xacro:include filename="$(find ovis_description)/urdf/ovis.urdf.xacro" />
     <xacro:include filename="$(find ovis_description)/urdf/kinova_common.xacro" />
-    <link name="base_link" />
-    <xacro:property name="robot_root" value="base_link" />
+    <link name="ovis_base_link" />
+    <xacro:property name="robot_root" value="ovis_base_link" />
     <xacro:ovis base_parent="${robot_root}" />
 </robot>

File: src/ovis_description/urdf/ovis_standalone.urdf.xacro (robot description, xacro)
@@ -3,10 +3,13 @@
     <xacro:include filename="$(find ovis_description)/urdf/gazebo.urdf.xacro" />
     <!-- <xacro:include filename="$(find ovis_description)/urdf/ovis.urdf.xacro" /> -->
-    <xacro:include filename="$(find ovis_description)/urdf/ovis2/urdf/ovis.urdf.xacro" />
+    <xacro:include
+        filename="$(find ovis_description)/urdf/ovis2/urdf/ovis.urdf.xacro" />
     <!-- <xacro:include filename="$(find ovis_description)/urdf/kinova_common.xacro" /> -->
-    <xacro:include filename="$(find ovis_description)/urdf/ovis2/urdf/ovis_common.xacro" />
-    <link name="world" />
+    <xacro:include
+        filename="$(find ovis_description)/urdf/ovis2/urdf/ovis_common.xacro" />
+    <xacro:property name="robot_root" value="ovis_base_link" />
+    <link name="base_link" />
     <!-- Define the base link -->
-    <link name="base_link">
+    <link name="ovis_base_link">
         <inertial>
             <origin xyz="0 0 0" />
@@ -15,11 +18,10 @@
         </inertial>
     </link>
-    <!-- Attach the base_link to the world with a fixed joint -->
+    <!-- Attach the ovis_base_link to the world or rove with a fixed joint -->
     <joint name="fixed_to_world" type="fixed">
-        <parent link="world" />
-        <child link="base_link" />
-        <origin xyz="0 0 0" rpy="0 0 0" />
+        <parent link="base_link" />
+        <child link="ovis_base_link" />
+        <origin xyz="-0.2 0 0.2" rpy="0 0 0" />
     </joint>
-    <xacro:property name="robot_root" value="base_link" />
     <xacro:ovis base_parent="${robot_root}" />
 </robot>

Commit message: Fix gazebo (#7)
* add moveit planing into gz

* add vcs for ros2 control gz

* force use sim tim on sim.launch.py

* add vcs to docker image

* add xacro if condition (gazebo, mock, real ovis)

* remove need for gazebo_config

* test ovis namespace

* fix errors and add controller namespace

* better node graph

* fix rviz2 trajectory issue

* remove namespace for joint state

* trajectory planner support with rove

File: src/ovis_description/urdf/gazebo.urdf.xacro (robot description, xacro)
@@ -1,24 +1,15 @@
 <?xml version="1.0"?>
 <robot xmlns:xacro="http://www.ros.org/wiki/xacro">
-    <xacro:macro name="gazebo_config" params="robot_namespace">
-        <!-- ros_control plugin -->
-        <gazebo>
-            <plugin name="gazebo_ros_control" filename="gz_ros_control.so">
-                <robotNamespace>${robot_namespace}</robotNamespace>
-                <robotSimType>gazebo_ros_control/DefaultRobotHWSim</robotSimType>
-                <legacyModeNS>true</legacyModeNS>
-            </plugin>
-        </gazebo>
-    </xacro:macro>
+    <!-- ros_control plugin -->
     <gazebo>
-        <plugin
-            filename="gz-sim-joint-state-publisher-system"
-            name="gz::sim::systems::JointStatePublisher">
-            <topic>joint_states</topic>
-        </plugin>
-        <plugin
-            filename="gz-sim-sensors-system"
-            name="gz::sim::systems::Sensors">
-            <render_engine>ogre2</render_engine>
+        <plugin filename="gz_ros2_control-system"
+            name="gz_ros2_control::GazeboSimROS2ControlPlugin">
+            <robot_param>robot_description</robot_param>
+            <robot_param_node>robot_state_publisher</robot_param_node>
+            <parameters>$(find ovis_moveit)/config/ros2_controllers.yaml</parameters>
+            <controller_manager_node_name>/ovis/controller_manager</controller_manager_node_name>
+            <ros>
+                <namespace>/ovis</namespace>
+            </ros>
         </plugin>
     </gazebo>

File: src/ovis_description/urdf/ovis_standalone.urdf.xacro (robot description, xacro)
@@ -3,9 +3,25 @@
     <xacro:include filename="$(find ovis_description)/urdf/gazebo.urdf.xacro" />
     <!-- <xacro:include filename="$(find ovis_description)/urdf/ovis.urdf.xacro" /> -->
-    <xacro:include filename="$(find ovis_description)/urdf/ovis2/urdf/ovis.urdf.xacro" />
+    <xacro:include
+        filename="$(find ovis_description)/urdf/ovis2/urdf/ovis.urdf.xacro" />
     <!-- <xacro:include filename="$(find ovis_description)/urdf/kinova_common.xacro" /> -->
-    <xacro:include filename="$(find ovis_description)/urdf/ovis2/urdf/ovis_common.xacro" />
+    <xacro:include
+        filename="$(find ovis_description)/urdf/ovis2/urdf/ovis_common.xacro" />
+    <xacro:property name="robot_root" value="ovis_base_link" />
     <link name="base_link" />
-    <xacro:property name="robot_root" value="base_link" />
+    <!-- Define the base link -->
+    <link name="ovis_base_link">
+        <inertial>
+            <origin xyz="0 0 0" />
+            <mass value="1.0" />
+            <inertia ixx="1.0" ixy="0.0" ixz="0.0" iyy="1.0" iyz="0.0" izz="1.0" />
+        </inertial>
+    </link>
+    <!-- Attach the ovis_base_link to the world or rove with a fixed joint -->
+    <joint name="fixed_to_world" type="fixed">
+        <parent link="base_link" />
+        <child link="ovis_base_link" />
+        <origin xyz="-0.2 0 0.2" rpy="0 0 0" />
+    </joint>
     <xacro:ovis base_parent="${robot_root}" />
 </robot>
