Commit message: cleaned up adn added ovis2 urdf

File: src/ovis_description/urdf/ovis2/urdf/ovis.urdf.xacro (robot description, xacro)
@@ -1,11 +1,11 @@
 <?xml version="1.0"?>
 <root xmlns:xacro="http://www.ros.org/wiki/xacro">
-    <xacro:property name="link_base_mesh" value="visual/ovis_base" />
-    <xacro:property name="link_1_mesh" value="visual/ovis_shoulder" />
-    <xacro:property name="link_2_mesh" value="visual/ovis_upper_arm" />
-    <xacro:property name="link_3_mesh" value="visual/ovis_elbow" />
-    <xacro:property name="link_4_mesh" value="visual/ovis_forearm" />
-    <xacro:property name="link_5_mesh" value="visual/ovis_wrist" />
-    <xacro:property name="link_6_mesh" value="visual/ovis_flange" />
+    <xacro:property name="link_base_mesh" value="ovis_base" />
+    <xacro:property name="link_1_mesh" value="ovis_j12" />
+    <xacro:property name="link_2_mesh" value="ovis_j23" />
+    <xacro:property name="link_3_mesh" value="ovis_j34" />
+    <xacro:property name="link_4_mesh" value="ovis_j45" />
+    <xacro:property name="link_5_mesh" value="ovis_j56" />
+    <xacro:property name="link_6_mesh" value="ovis_end_effector" />
     <xacro:property name="link_base_mesh_no" value="0" />
     <xacro:property name="link_1_mesh_no" value="1" />
@@ -20,9 +20,9 @@
     <!-- Transferred to a parameter in the ovis macro -->
     <!-- <xacro:property name="joint_base_origin_xyz" value="0 0 0" /> -->
-    <xacro:property name="joint_base_origin_rpy" value="${J_PI/2} 0 0" />
+    <xacro:property name="joint_base_origin_rpy" value="0 0 0" />
     <xacro:property name="joint_1" value="joint_1" />
     <xacro:property name="joint_1_type" value="continuous" />
-    <xacro:property name="joint_1_axis_xyz" value="0 1 0" />
-    <xacro:property name="joint_1_origin_xyz" value="0 0.051 0" />
+    <xacro:property name="joint_1_axis_xyz" value="0 0 1" />
+    <xacro:property name="joint_1_origin_xyz" value="0 0 0.03" />
     <xacro:property name="joint_1_origin_rpy" value="0 0 0" />
     <xacro:property name="joint_1_lower_limit" value="${-4*J_PI}" />
@@ -32,17 +32,17 @@
     <xacro:property name="joint_2" value="joint_2" />
     <xacro:property name="joint_2_type" value="revolute" />
-    <xacro:property name="joint_2_axis_xyz" value="0 0 1" />
-    <xacro:property name="joint_2_origin_xyz" value="0 0.0889 0" />
-    <xacro:property name="joint_2_origin_rpy" value="0 0 ${-J_PI/2}" />
-    <xacro:property name="joint_2_lower_limit" value="0" />
-    <xacro:property name="joint_2_upper_limit" value="${J_PI}" />
+    <xacro:property name="joint_2_axis_xyz" value="0 1 0" />
+    <xacro:property name="joint_2_origin_xyz" value="0.00004 0.0625 0.07001" />
+    <xacro:property name="joint_2_origin_rpy" value="0 0 0" />
+    <xacro:property name="joint_2_lower_limit" value="-3.40339" />
+    <xacro:property name="joint_2_upper_limit" value="0.26180" />
     <xacro:property name="joint_2_velocity_limit" value="${36*J_PI/180}" />
     <xacro:property name="joint_2_torque_limit" value="80" />
     <xacro:property name="joint_3" value="joint_3" />
     <xacro:property name="joint_3_type" value="revolute" />
-    <xacro:property name="joint_3_axis_xyz" value="0 0 1" />
-    <xacro:property name="joint_3_origin_xyz" value="0 0.465 0" />
-    <xacro:property name="joint_3_origin_rpy" value="0 0 ${J_PI}" />
-    <xacro:property name="joint_3_lower_limit" value="${-J_PI}" />
+    <xacro:property name="joint_3_axis_xyz" value="0 -1 0" />
+    <xacro:property name="joint_3_origin_xyz" value="0.30039 -0.01763 0.00072" />
+    <xacro:property name="joint_3_origin_rpy" value="0 0 0" />
+    <xacro:property name="joint_3_lower_limit" value="-5.23599" />
     <xacro:property name="joint_3_upper_limit" value="0" />
     <xacro:property name="joint_3_velocity_limit" value="${36*J_PI/180}" />
@@ -50,6 +50,6 @@
     <xacro:property name="joint_4" value="joint_4" />
     <xacro:property name="joint_4_type" value="continuous" />
-    <xacro:property name="joint_4_axis_xyz" value="0 1 0" />
-    <xacro:property name="joint_4_origin_xyz" value="0.0889 0.047625 0" />
+    <xacro:property name="joint_4_axis_xyz" value="-1 0 0" />
+    <xacro:property name="joint_4_origin_xyz" value="-0.06672 -0.04897 -0.00044" />
     <xacro:property name="joint_4_origin_rpy" value="0 0 0" />
     <xacro:property name="joint_4_lower_limit" value="${-4*J_PI}" />
@@ -59,16 +59,16 @@
     <xacro:property name="joint_5" value="joint_5" />
     <xacro:property name="joint_5_type" value="revolute" />
-    <xacro:property name="joint_5_axis_xyz" value="0 0 1" />
-    <xacro:property name="joint_5_origin_xyz" value="0 0.265 0" />
+    <xacro:property name="joint_5_axis_xyz" value="0 1 0" />
+    <xacro:property name="joint_5_origin_xyz" value="-0.33480 0.00015 0.00051" />
     <xacro:property name="joint_5_origin_rpy" value="0 0 0" />
-    <xacro:property name="joint_5_lower_limit" value="${-J_PI/2}" />
-    <xacro:property name="joint_5_upper_limit" value="${J_PI/2}" />
+    <xacro:property name="joint_5_lower_limit" value="-1.65806" />
+    <xacro:property name="joint_5_upper_limit" value="1.65806" />
     <xacro:property name="joint_5_velocity_limit" value="${48*J_PI/180}" />
     <xacro:property name="joint_5_torque_limit" value="20" />
     <xacro:property name="joint_6" value="joint_6" />
     <xacro:property name="joint_6_type" value="continuous" />
-    <xacro:property name="joint_6_axis_xyz" value="0 0 1" />
-    <xacro:property name="joint_6_origin_xyz" value="0 0.0762 0" />
-    <xacro:property name="joint_6_origin_rpy" value="${J_PI/2} ${J_PI/2} 0" />
+    <xacro:property name="joint_6_axis_xyz" value="-1 0 0" />
+    <xacro:property name="joint_6_origin_xyz" value="-0.07 0.00003 0.00001" />
+    <xacro:property name="joint_6_origin_rpy" value="0 0 0" />
     <!-- If gripper inverted, use this line instead -->
     <!-- <xacro:property name="joint_6_origin_rpy" value="$${-J_PI/3} 0 0" /> -->
@@ -82,5 +82,5 @@
     <xacro:property name="joint_end_effector_origin_xyz" value="0 0 -0.1600" />
     <xacro:property name="joint_end_effector_origin_rpy" value="${J_PI} 0 ${J_PI/2}" />
-    <xacro:macro name="ovis" params="base_parent type:=ovis prefix:=ovis joint_base_origin_xyz:='0 0 0'">
+    <xacro:macro name="ovis" params="base_parent prefix:=ovis joint_base_origin_xyz:='0 0 0'">
         <xacro:gazebo_config robot_namespace="${prefix}" />
         <xacro:kinova_armlink link_name="${prefix}_link_base" link_mesh="${link_base_mesh}"

File: src/ovis_description/urdf/ovis_standalone.urdf.xacro (robot description, xacro)
@@ -2,6 +2,8 @@
 <robot name="ovis" xmlns:xacro="http://www.ros.org/wiki/xacro">
     <xacro:include filename="$(find ovis_description)/urdf/gazebo.urdf.xacro" />
-    <xacro:include filename="$(find ovis_description)/urdf/ovis.urdf.xacro" />
-    <xacro:include filename="$(find ovis_description)/urdf/kinova_common.xacro" />
+    <!-- <xacro:include filename="$(find ovis_description)/urdf/ovis.urdf.xacro" /> -->
+    <xacro:include filename="$(find ovis_description)/urdf/ovis2/urdf/ovis.urdf.xacro" />
+    <!-- <xacro:include filename="$(find ovis_description)/urdf/kinova_common.xacro" /> -->
+    <xacro:include filename="$(find ovis_description)/urdf/ovis2/urdf/ovis_common.xacro" />
     <link name="base_link" />
     <xacro:property name="robot_root" value="base_link" />

File: src/ovis_moveit/config/ovis.ros2_control.xacro (robot description, xacro)
@@ -9,5 +9,5 @@
                 <plugin>ovis_control/OvisHWInterface</plugin>
                 <param name="api_type">ETHERNET</param>
-                <!-- USB or ETHERNET-->
+                <!-- USB or ETHERNET -->
                 <param name="local_machine_IP">192.168.84.15</param>
                 <param name="subnet_mask">255.255.255.0</param>
@@ -19,4 +19,5 @@
             <joint name="ovis_joint_1">
                 <command_interface name="position"/>
+                <command_interface name="velocity"/>
                 <state_interface name="position">
                   <!-- <param name="initial_value">${initial_positions['ovis_joint_1']}</param> -->
@@ -25,5 +26,6 @@
             </joint>
             <joint name="ovis_joint_2">
-                <command_interface name="position"/>
+              <command_interface name="position"/>
+              <command_interface name="velocity"/>
                 <state_interface name="position">
                   <!-- <param name="initial_value">${initial_positions['ovis_joint_2']}</param> -->
@@ -33,4 +35,5 @@
             <joint name="ovis_joint_3">
                 <command_interface name="position"/>
+                <command_interface name="velocity"/>
                 <state_interface name="position">
                   <!-- <param name="initial_value">${initial_positions['ovis_joint_3']}</param> -->
@@ -40,4 +43,5 @@
             <joint name="ovis_joint_4">
                 <command_interface name="position"/>
+                <command_interface name="velocity"/>
                 <state_interface name="position">
                   <!-- <param name="initial_value">${initial_positions['ovis_joint_4']}</param> -->
@@ -47,4 +51,5 @@
             <joint name="ovis_joint_5">
                 <command_interface name="position"/>
+                <command_interface name="velocity"/>
                 <state_interface name="position">
                   <!-- <param name="initial_value">${initial_positions['ovis_joint_5']}</param> -->
@@ -54,4 +59,5 @@
             <joint name="ovis_joint_6">
                 <command_interface name="position"/>
+                <command_interface name="velocity"/>
                 <state_interface name="position">
                   <!-- <param name="initial_value">${initial_positions['ovis_joint_6']}</param> -->

Commit message: changed end effector marker position and zero position of motors

File: src/ovis_description/urdf/ovis2/urdf/ovis.urdf.xacro (robot description, xacro)
@@ -80,5 +80,5 @@
     <xacro:property name="joint_end_effector_type" value="fixed" />
     <xacro:property name="joint_end_effector_axis_xyz" value="0 0 0" />
-    <xacro:property name="joint_end_effector_origin_xyz" value="0 0 -0.1600" />
+    <xacro:property name="joint_end_effector_origin_xyz" value="-0.25 0 0" />
     <xacro:property name="joint_end_effector_origin_rpy" value="${J_PI} 0 ${J_PI/2}" />
     <xacro:macro name="ovis" params="base_parent prefix:=ovis joint_base_origin_xyz:='0 0 0'">
