Commit message: cleaned code and automatic launch file ovis_bringup combined.launch.py

File: src/ovis_description/urdf/ovis2/urdf/ovis2.urdf (robot description, URDF)
Before this commit: robot ovis2, 7 links, 6 joints
Links:
- link ovis2_base_link: geometry collision mesh filename=package://ovis_description/urdf/ovis2/meshes/collision/ovis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 scale=1 1 1; visual mesh filename=package://ovis_description/urdf/ovis2/meshes/collision/ovis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 scale=1 1 1
- link ovis2_link_1: geometry collision mesh filename=package://ovis_description/urdf/ovis2/meshes/collision/ovis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 scale=1 1 1; visual mesh filename=package://ovis_description/urdf/ovis2/meshes/collision/ovis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 scale=1 1 1
- link ovis2_link_2: geometry collision mesh filename=package://ovis_description/urdf/ovis2/meshes/collision/ovis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 scale=1 1 1; visual mesh filename=package://ovis_description/urdf/ovis2/meshes/collision/ovis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 scale=1 1 1
- link ovis2_link_3: geometry collision mesh filename=package://ovis_description/urdf/ovis2/meshes/collision/ovis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 scale=1 1 1; visual mesh filename=package://ovis_description/urdf/ovis2/meshes/collision/ovis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 scale=1 1 1
- link ovis2_link_4: geometry collision mesh filename=package://ovis_description/urdf/ovis2/meshes/collision/ovis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 scale=1 1 1; visual mesh filename=package://ovis_description/urdf/ovis2/meshes/collision/ovis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 scale=1 1 1
- link ovis2_link_5: geometry collision mesh filename=package://ovis_description/urdf/ovis2/meshes/collision/ovis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 scale=1 1 1; visual mesh filename=package://ovis_description/urdf/ovis2/meshes/collision/ovis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 scale=1 1 1
- link ovis2_link_6: geometry collision mesh filename=package://ovis_description/urdf/ovis2/meshes/collision/ovis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 scale=1 1 1; visual mesh filename=package://ovis_description/urdf/ovis2/meshes/collision/ovis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 scale=1 1 1

File: src/ovis_description/urdf/ovis2/urdf/ovis_common.xacro (robot description, xacro)
@@ -19,6 +19,5 @@
             <visual name="${link_name}_vis">
                 <geometry>
-                    <mesh
-                        filename="file://$(find ovis_description)/urdf/ovis2/meshes/visual/${link_mesh}.stl"/>
+                    <mesh filename="package://ovis_description/urdf/ovis2/meshes/visual/${link_mesh}.stl"/>
                 </geometry>
                 <material name="carbon_fiber">
@@ -28,14 +27,13 @@
             <collision name="${link_name}_col">
                 <geometry>
-                    <mesh
-                        filename="$(find ovis_description)/urdf/ovis2/meshes/collision/${link_mesh}.stl"/>
+                    <mesh filename="package://ovis_description/urdf/ovis2/meshes/collision/${link_mesh}.stl"/>
                 </geometry>
             </collision>
-						<inertial>
-              <inertia ixx="0.00001" ixy="0.00000" ixz="0.00000" iyy="0.00001" iyz="0.00000" izz="0.00001"/>
-              <origin rpy="0.00000 0.00000 0.00000" xyz="0.00000 0.00000 0.00000"/>
-              <mass value="0.1"/>
+            <inertial>
+                <inertia ixx="0.00001" ixy="0.00000" ixz="0.00000" iyy="0.00001" iyz="0.00000" izz="0.00001"/>
+                <origin rpy="0.00000 0.00000 0.00000" xyz="0.00000 0.00000 0.00000"/>
+                <mass value="0.1"/>
             </inertial>
-      </link>
+        </link>
     </xacro:macro>
   <!--

Commit message: change to something gazebo can see

File: src/ovis_description/urdf/ovis2/urdf/ovis2.urdf (robot description, URDF)
Before this commit: robot ovis2, 7 links, 6 joints
Links:
- link ovis2_base_link: geometry collision mesh filename=file://$(find ovis_description)/urdf/ovis2/meshes/collision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 scale=1 1 1; visual mesh filename=file://$(find ovis_description)/urdf/ovis2/meshes/collision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 scale=1 1 1
- link ovis2_link_1: geometry collision mesh filename=file://$(find ovis_description)/urdf/ovis2/meshes/collision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 scale=1 1 1; visual mesh filename=file://$(find ovis_description)/urdf/ovis2/meshes/collision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 scale=1 1 1
- link ovis2_link_2: geometry collision mesh filename=file://$(find ovis_description)/urdf/ovis2/meshes/collision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 scale=1 1 1; visual mesh filename=file://$(find ovis_description)/urdf/ovis2/meshes/collision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 scale=1 1 1
- link ovis2_link_3: geometry collision mesh filename=file://$(find ovis_description)/urdf/ovis2/meshes/collision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 scale=1 1 1; visual mesh filename=file://$(find ovis_description)/urdf/ovis2/meshes/collision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 scale=1 1 1
- link ovis2_link_4: geometry collision mesh filename=file://$(find ovis_description)/urdf/ovis2/meshes/collision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 scale=1 1 1; visual mesh filename=file://$(find ovis_description)/urdf/ovis2/meshes/collision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 scale=1 1 1
- link ovis2_link_5: geometry collision mesh filename=file://$(find ovis_description)/urdf/ovis2/meshes/collision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 scale=1 1 1; visual mesh filename=file://$(find ovis_description)/urdf/ovis2/meshes/collision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 scale=1 1 1
- link ovis2_link_6: geometry collision mesh filename=file://$(find ovis_description)/urdf/ovis2/meshes/collision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 scale=1 1 1; visual mesh filename=file://$(find ovis_description)/urdf/ovis2/meshes/collision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 scale=1 1 1

File: src/ovis_description/urdf/ovis2/urdf/ovis_common.xacro (robot description, xacro)
@@ -19,5 +19,5 @@
             <visual name="${link_name}_vis">
                 <geometry>
-                    <mesh filename="package://ovis_description/urdf/ovis2/meshes/visual/${link_mesh}.stl"/>
+                    <mesh filename="file://$(find ovis_description)/urdf/ovis2/meshes/visual/${link_mesh}.stl"/>
                 </geometry>
                 <material name="carbon_fiber">
@@ -27,5 +27,5 @@
             <collision name="${link_name}_col">
                 <geometry>
-                    <mesh filename="package://ovis_description/urdf/ovis2/meshes/collision/${link_mesh}.stl"/>
+                    <mesh filename="file://$(find ovis_description)/urdf/ovis2/meshes/collision/${link_mesh}.stl"/>
                 </geometry>
             </collision>
