Commit message: Almost working

File: src/ovis_moveit/config/ovis.ros2_control.xacro (robot description, xacro)
@@ -2,5 +2,5 @@
 <robot xmlns:xacro="http://www.ros.org/wiki/xacro">
     <xacro:macro name="ovis_ros2_control" params="name initial_positions_file">
-        <xacro:property name="initial_positions" value="${load_yaml(initial_positions_file)['initial_positions']}"/>
+        <xacro:property name="initial_positions" value="${xacro.load_yaml(initial_positions_file)['initial_positions']}"/>
         <ros2_control name="${name}" type="system">
             <hardware>
@@ -8,6 +8,7 @@
                 <!-- <plugin>mock_components/GenericSystem</plugin> -->
                 <plugin>ovis_control/OvisHWInterface</plugin>
-                <param name="api_type">ETHERNET</param> <!-- USB or ETHERNET-->
-                <param name="local_machine_ip">192.168.84.15</param>
+                <param name="api_type">ETHERNET</param>
+                <!-- USB or ETHERNET-->
+                <param name="local_machine_IP">192.168.84.15</param>
                 <param name="subnet_mask">255.255.255.0</param>
                 <param name="local_cmd_port">25015</param>
@@ -19,5 +20,5 @@
                 <command_interface name="position"/>
                 <state_interface name="position">
-                  <param name="initial_value">${initial_positions['ovis_joint_1']}</param>
+                  <!-- <param name="initial_value">${initial_positions['ovis_joint_1']}</param> -->
                 </state_interface>
                 <state_interface name="velocity"/>
@@ -26,5 +27,5 @@
                 <command_interface name="position"/>
                 <state_interface name="position">
-                  <param name="initial_value">${initial_positions['ovis_joint_2']}</param>
+                  <!-- <param name="initial_value">${initial_positions['ovis_joint_2']}</param> -->
                 </state_interface>
                 <state_interface name="velocity"/>
@@ -33,5 +34,5 @@
                 <command_interface name="position"/>
                 <state_interface name="position">
-                  <param name="initial_value">${initial_positions['ovis_joint_3']}</param>
+                  <!-- <param name="initial_value">${initial_positions['ovis_joint_3']}</param> -->
                 </state_interface>
                 <state_interface name="velocity"/>
@@ -40,5 +41,5 @@
                 <command_interface name="position"/>
                 <state_interface name="position">
-                  <param name="initial_value">${initial_positions['ovis_joint_4']}</param>
+                  <!-- <param name="initial_value">${initial_positions['ovis_joint_4']}</param> -->
                 </state_interface>
                 <state_interface name="velocity"/>
@@ -47,5 +48,5 @@
                 <command_interface name="position"/>
                 <state_interface name="position">
-                  <param name="initial_value">${initial_positions['ovis_joint_5']}</param>
+                  <!-- <param name="initial_value">${initial_positions['ovis_joint_5']}</param> -->
                 </state_interface>
                 <state_interface name="velocity"/>
@@ -54,5 +55,5 @@
                 <command_interface name="position"/>
                 <state_interface name="position">
-                  <param name="initial_value">${initial_positions['ovis_joint_6']}</param>
+                  <!-- <param name="initial_value">${initial_positions['ovis_joint_6']}</param> -->
                 </state_interface>
                 <state_interface name="velocity"/>

Commit message: add xacro if condition (gazebo, mock, real ovis)

File: src/ovis_moveit/config/ovis.ros2_control.xacro (robot description, xacro)
@@ -1,64 +1,69 @@
 <?xml version="1.0"?>
 <robot xmlns:xacro="http://www.ros.org/wiki/xacro">
-    <xacro:macro name="ovis_ros2_control" params="name initial_positions_file">
-        <xacro:property name="initial_positions" value="${xacro.load_yaml(initial_positions_file)['initial_positions']}"/>
-        <ros2_control name="${name}" type="system">
-            <hardware>
-                <!-- By default, set up controllers for simulation. This won't work on real hardware -->
-                <plugin>gz_ros2_control/GazeboSimSystem</plugin>
-                <!-- Old plugin that work without gazebo -->
-                <!-- <plugin>mock_components/GenericSystem</plugin> -->
-                <!-- <plugin>ovis_control/OvisHWInterface</plugin> -->
-                <!-- USB or ETHERNET -->
-                <!-- <param name="api_type">ETHERNET</param>
-                <param name="local_machine_IP">192.168.84.15</param>
-                <param name="subnet_mask">255.255.255.0</param>
-                <param name="local_cmd_port">25015</param>
-                <param name="local_broadcast_port">25025</param>
-                <param name="robot_ip_address">192.168.84.160</param> -->
-            </hardware>
-            <joint name="ovis_joint_1">
-                <command_interface name="position"/>
-                <state_interface name="position">
-                  <param name="initial_value">${initial_positions['ovis_joint_1']}</param>
-                </state_interface>
-                <state_interface name="velocity"/>
-            </joint>
-            <joint name="ovis_joint_2">
-                <command_interface name="position"/>
-                <state_interface name="position">
-                  <param name="initial_value">${initial_positions['ovis_joint_2']}</param>
-                </state_interface>
-                <state_interface name="velocity"/>
-            </joint>
-            <joint name="ovis_joint_3">
-                <command_interface name="position"/>
-                <state_interface name="position">
-                  <param name="initial_value">${initial_positions['ovis_joint_3']}</param>
-                </state_interface>
-                <state_interface name="velocity"/>
-            </joint>
-            <joint name="ovis_joint_4">
-                <command_interface name="position"/>
-                <state_interface name="position">
-                  <param name="initial_value">${initial_positions['ovis_joint_4']}</param>
-                </state_interface>
-                <state_interface name="velocity"/>
-            </joint>
-            <joint name="ovis_joint_5">
-                <command_interface name="position"/>
-                <state_interface name="position">
-                  <param name="initial_value">${initial_positions['ovis_joint_5']}</param>
-                </state_interface>
-                <state_interface name="velocity"/>
-            </joint>
-            <joint name="ovis_joint_6">
-                <command_interface name="position"/>
-                <state_interface name="position">
-                  <param name="initial_value">${initial_positions['ovis_joint_6']}</param>
-                </state_interface>
-                <state_interface name="velocity"/>
-            </joint>
-        </ros2_control>
-    </xacro:macro>
+  <xacro:macro name="ovis_ros2_control" params="name initial_positions_file hardware_type">
+    <xacro:property name="initial_positions"
+      value="${xacro.load_yaml(initial_positions_file)['initial_positions']}" />
+    <ros2_control name="${name}" type="system">
+      <hardware>
+        <xacro:if value="${hardware_type == 'gazebo'}">
+          <plugin>gz_ros2_control/GazeboSimSystem</plugin>
+        </xacro:if>
+        <xacro:if value="${hardware_type == 'mock'}">
+          <plugin>mock_components/GenericSystem</plugin>
+        </xacro:if>
+        <xacro:if value="${hardware_type == 'ovis'}">
+          <plugin>ovis_control/OvisHWInterface</plugin>
+          <param name="api_type">ETHERNET</param>
+          <param name="local_machine_IP">192.168.84.15</param>
+          <param name="subnet_mask">255.255.255.0</param>
+          <param name="local_cmd_port">25015</param>
+          <param name="local_broadcast_port">25025</param>
+          <param name="robot_ip_address">192.168.84.160</param>
+        </xacro:if>
+      </hardware>
+      <!-- Define joints here -->
+      <joint name="ovis_joint_1">
+        <command_interface name="position" />
+        <state_interface name="position">
+          <param name="initial_value">${initial_positions['ovis_joint_1']}</param>
+        </state_interface>
+        <state_interface name="velocity" />
+      </joint>
+      <joint name="ovis_joint_2">
+        <command_interface name="position" />
+        <state_interface name="position">
+          <param name="initial_value">${initial_positions['ovis_joint_2']}</param>
+        </state_interface>
+        <state_interface name="velocity" />
+      </joint>
+      <joint name="ovis_joint_3">
+        <command_interface name="position" />
+        <state_interface name="position">
+          <param name="initial_value">${initial_positions['ovis_joint_3']}</param>
+        </state_interface>
+        <state_interface name="velocity" />
+      </joint>
+      <joint name="ovis_joint_4">
+        <command_interface name="position" />
+        <state_interface name="position">
+          <param name="initial_value">${initial_positions['ovis_joint_4']}</param>
+        </state_interface>
+        <state_interface name="velocity" />
+      </joint>
+      <joint name="ovis_joint_5">
+        <command_interface name="position" />
+        <state_interface name="position">
+          <param name="initial_value">${initial_positions['ovis_joint_5']}</param>
+        </state_interface>
+        <state_interface name="velocity" />
+      </joint>
+      <joint name="ovis_joint_6">
+        <command_interface name="position" />
+        <state_interface name="position">
+          <param name="initial_value">${initial_positions['ovis_joint_6']}</param>
+        </state_interface>
+        <state_interface name="velocity" />
+      </joint>
+    </ros2_control>
+  </xacro:macro>
 </robot>
