Commit message: Refactoring for ovis 2

File: src/ovis_description/urdf/ovis2/kinova_common.xacro (robot description, xacro)
@@ -13,11 +13,12 @@
     xmlns:physics="http://playerstage.sourceforge.net/gazebo/xmlschema/#physics"
 	xmlns:xacro="http://www.ros.org/wiki/xacro">
-<!-- <xacro:include filename="$(find ovis_description)/urdf/kinova_inertial.xacro" /> -->
+<xacro:include filename="$(find ovis_description)/urdf/ovis2/kinova_inertial.xacro" />
     <xacro:property name="J_PI" value="3.1415926535897931" />
     <xacro:macro name="kinova_armlink" params="link_name link_mesh ring_mesh:=ring_big use_ring_mesh:=false mesh_no">
         <link name="${link_name}">
-            <visual name="${link_name}_vis">
+            <visual>
                 <geometry>
-                    <mesh filename="file://$(find ovis_description)/urdf/ovis2/meshes/visual/${link_mesh}.stl"/>
+                    <mesh
+                        filename="file://$(find ovis_description)/meshes/ovis2/${link_mesh}.stl"/>
                 </geometry>
                 <material name="carbon_fiber">
@@ -25,15 +26,21 @@
                 </material>
             </visual>
-            <collision name="${link_name}_col">
+	    <!-- Adding ring to the model -->
+	         <xacro:if value="${use_ring_mesh}">
+	           <visual>
                 <geometry>
-                    <mesh filename="file://$(find ovis_description)/urdf/ovis2/meshes/collision/${link_mesh}.stl"/>
+                    <mesh
+                        filename="$(find ovis_description)/meshes/ovis2/${ring_mesh}.stl"/>
+                </geometry>
+             </visual>
+	    </xacro:if>
+            <collision>
+                <geometry>
+                    <mesh
+                        filename="$(find ovis_description)/meshes/ovis2/${link_mesh}.stl"/>
                 </geometry>
             </collision>
-            <inertial>
-                <inertia ixx="0.00001" ixy="0.00000" ixz="0.00000" iyy="0.00001" iyz="0.00000" izz="0.00001"/>
-                <origin rpy="0.00000 0.00000 0.00000" xyz="0.00000 0.00000 0.00000"/>
-                <mass value="0.1"/>
-            </inertial>
-        </link>
+						<xacro:kinova_inertial mesh_no="${mesh_no}"/>
+      </link>
     </xacro:macro>
   <!--
@@ -96,5 +103,5 @@
       </gazebo>
       <gazebo>
-        <plugin filename="gz-sim-forcetorque-system" name="gz::sim::systems::ForceTorque">
+        <plugin name="gz::sim::systems::ForceTorque" filename="gz-sim-forcetorque-system">
           <updateRate>30.0</updateRate>
           <topicName>${joint_name}_ft_sensor_topic</topicName>

File: src/ovis_description/urdf/ovis2/ovis.urdf.xacro (robot description, xacro)
@@ -1,4 +1,5 @@
 <?xml version="1.0"?>
 <root xmlns:xacro="http://www.ros.org/wiki/xacro">
+    <xacro:include filename="$(find ovis_description)/urdf/ovis2/ovis_common.xacro" />
     <xacro:property name="link_base_mesh" value="ovis_base" />
     <xacro:property name="link_1_mesh" value="ovis_j12" />

File: src/ovis_description/urdf/ovis2/ovis2.urdf (robot description, URDF)
Before this commit: robot ovis2, 7 links, 6 joints
Links:
- link ovis2_base_link: geometry collision mesh filename=file://$(find ovis_description)/meshes/ovis2/collision/ovis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 scale=1 1 1; visual mesh filename=file://$(find ovis_description)/meshes/ovis2/collision/ovis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 scale=1 1 1
- link ovis2_link_1: geometry collision mesh filename=file://$(find ovis_description)/meshes/ovis2/collision/ovis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 scale=1 1 1; visual mesh filename=file://$(find ovis_description)/meshes/ovis2/collision/ovis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 scale=1 1 1
- link ovis2_link_2: geometry collision mesh filename=file://$(find ovis_description)/meshes/ovis2/collision/ovis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 scale=1 1 1; visual mesh filename=file://$(find ovis_description)/meshes/ovis2/collision/ovis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 scale=1 1 1
- link ovis2_link_3: geometry collision mesh filename=file://$(find ovis_description)/meshes/ovis2/collision/ovis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 scale=1 1 1; visual mesh filename=file://$(find ovis_description)/meshes/ovis2/collision/ovis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 scale=1 1 1
- link ovis2_link_4: geometry collision mesh filename=file://$(find ovis_description)/meshes/ovis2/collision/ovis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 scale=1 1 1; visual mesh filename=file://$(find ovis_description)/meshes/ovis2/collision/ovis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 scale=1 1 1
- link ovis2_link_5: geometry collision mesh filename=file://$(find ovis_description)/meshes/ovis2/collision/ovis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 scale=1 1 1; visual mesh filename=file://$(find ovis_description)/meshes/ovis2/collision/ovis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 scale=1 1 1
- link ovis2_link_6: geometry collision mesh filename=file://$(find ovis_description)/meshes/ovis2/collision/ovis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 scale=1 1 1; visual mesh filename=file://$(find ovis_description)/meshes/ovis2/collision/ovis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 scale=1 1 1

File: src/ovis_description/urdf/ovis2/ovis_common.xacro (robot description, xacro)
@@ -13,12 +13,11 @@
     xmlns:physics="http://playerstage.sourceforge.net/gazebo/xmlschema/#physics"
 	xmlns:xacro="http://www.ros.org/wiki/xacro">
-<xacro:include filename="$(find ovis_description)/urdf/kinova_inertial.xacro" />
+<!-- <xacro:include filename="$(find ovis_description)/urdf/kinova_inertial.xacro" /> -->
     <xacro:property name="J_PI" value="3.1415926535897931" />
     <xacro:macro name="kinova_armlink" params="link_name link_mesh ring_mesh:=ring_big use_ring_mesh:=false mesh_no">
         <link name="${link_name}">
-            <visual>
+            <visual name="${link_name}_vis">
                 <geometry>
-                    <mesh
-                        filename="file://$(find ovis_description)/meshes/${link_mesh}.stl"/>
+                    <mesh filename="file://$(find ovis_description)/meshes/ovis2/visual/${link_mesh}.stl"/>
                 </geometry>
                 <material name="carbon_fiber">
@@ -26,21 +25,15 @@
                 </material>
             </visual>
-	    <!-- Adding ring to the model -->
-	         <xacro:if value="${use_ring_mesh}">
-	           <visual>
+            <collision name="${link_name}_col">
                 <geometry>
-                    <mesh
-                        filename="$(find ovis_description)/meshes/${ring_mesh}.stl"/>
-                </geometry>
-             </visual>
-	    </xacro:if>
-            <collision>
-                <geometry>
-                    <mesh
-                        filename="$(find ovis_description)/meshes/${link_mesh}.stl"/>
+                    <mesh filename="file://$(find ovis_description)/meshes/ovis2/collision/${link_mesh}.stl"/>
                 </geometry>
             </collision>
-						<xacro:kinova_inertial mesh_no="${mesh_no}"/>
-      </link>
+            <inertial>
+                <inertia ixx="0.00001" ixy="0.00000" ixz="0.00000" iyy="0.00001" iyz="0.00000" izz="0.00001"/>
+                <origin rpy="0.00000 0.00000 0.00000" xyz="0.00000 0.00000 0.00000"/>
+                <mass value="0.1"/>
+            </inertial>
+        </link>
     </xacro:macro>
   <!--
@@ -103,5 +96,5 @@
       </gazebo>
       <gazebo>
-        <plugin name="gz::sim::systems::ForceTorque" filename="gz-sim-forcetorque-system">
+        <plugin filename="gz-sim-forcetorque-system" name="gz::sim::systems::ForceTorque">
           <updateRate>30.0</updateRate>
           <topicName>${joint_name}_ft_sensor_topic</topicName>

File: src/ovis_moveit/config/ovis.ros2_control.xacro (robot description, xacro)
@@ -12,5 +12,5 @@
           <plugin>mock_components/GenericSystem</plugin>
         </xacro:if>
-        <xacro:if value="${hardware_type == 'ovis'}">
+        <xacro:if value="${hardware_type == 'real'}">
           <plugin>ovis_control/OvisHWInterface</plugin>
           <param name="api_type">ETHERNET</param>

File: src/ovis_moveit/config/ovis.urdf.xacro (robot description, xacro)
@@ -2,7 +2,8 @@
 <robot xmlns:xacro="http://www.ros.org/wiki/xacro" name="ovis">
     <xacro:arg name="initial_positions_file" default="initial_positions.yaml" />
-    <xacro:arg name="hardware_type" default="ovis" />
+    <xacro:arg name="hardware_type" default="real" />
+    <xacro:arg name="version" default="ovis2" />
     <!-- Import ovis urdf file -->
-    <xacro:include filename="$(find ovis_description)/urdf/ovis_standalone.urdf.xacro" />
+    <xacro:include filename="$(find ovis_description)/urdf/$(version)/ovis_standalone.urdf.xacro"/>
     <!-- Import control_xacro -->
     <xacro:include filename="ovis.ros2_control.xacro" />
